Commit message: update

File: motion-planning-sim/Assets/Robots/MobileManipulator/urdf/mobile_manipulator.urdf (robot description, URDF)
Before this commit: robot mobile_manipulator, 17 links, 16 joints
Links:
- added link livox_frame
Joints:
- added joint livox_joint: type fixed, parent top_sensor_mount_link, child livox_frame, origin xyz=0 0 0.047 rpy=0 0 0

File: ros2_ws/src/mobile_manipulator_description/urdf/mobile_manipulator.urdf (robot description, URDF)
Before this commit: robot mobile_manipulator, 17 links, 16 joints
Links:
- added link livox_frame
Joints:
- added joint livox_joint: type fixed, parent top_sensor_mount_link, child livox_frame, origin xyz=0 0 0.047 rpy=0 0 0

Commit message: initial setup and tests

File: motion-planning-sim/Assets/Robots/MobileManipulator/urdf/mobile_manipulator.urdf (robot description, URDF)
Before this commit: robot mobile_manipulator, 18 links, 17 joints
Joints:
- joint shoulder_lift_joint: limit lower=-1.74532925199 upper=1.74532925199 effort=120 velocity=1.6 -> lower=-1.74532925199 upper=1.74532925199 effort=160 velocity=1.6

File: ros2_ws/src/mobile_manipulator_description/urdf/mobile_manipulator.urdf (robot description, URDF)
Before this commit: robot mobile_manipulator, 18 links, 17 joints
Joints:
- joint shoulder_lift_joint: limit lower=-1.74532925199 upper=1.74532925199 effort=120 velocity=1.6 -> lower=-1.74532925199 upper=1.74532925199 effort=160 velocity=1.6
